File: Hardware/FOC_Driver/MCU_sch.kicad_sch (KiCad schematic)
At the start: 1 part, among them U1 STM32G431CBUx

Commit message: Schematic update and Firmware folder
Parts:
- added C25, C26, C32, C33, C36, C38, C9: 100n, symbol Device:C
- added C27, C28: 15p, symbol Device:C
- added C29, C30, C31: 2n2, symbol Device:C
- added C34: 1u, symbol Device:C
- added C35: 4u7, symbol Device:C
- added D4, D5: LED, symbol Device:LED
- added FB1: FerriteBead, symbol Device:FerriteBead
- added R22: 10k, symbol Device:R
- added R23, R24: 1k, symbol Device:R
- added R25, R26, R27: 100, symbol Device:R
- added Y1: 8Mhz, symbol Device:Crystal_GND24
Connections:
- net +3V3: now reaches U1.1 (VBAT)
- net +3V3: now also U1.23 (VDD), U1.35 (VDD), U1.48 (VDD), C25.2, C26.2, C32.2, C35.2, C9.2, FB1.2
- net at U1.10 (PA2): now also C31.2, R27.1
- net VBAT_SENSE: now reaches U1.11 (PA3)
- net ENC_CS: now reaches U1.12 (PA4)
- net ENC_SCK: now reaches U1.13 (PA5)
- net ENC_MISO: now reaches U1.14 (PA6)
- net ENC_MOSI: now reaches U1.15 (PA7)
- net +3V3A: now reaches U1.20 (VREF+)
- net +3V3A: now also U1.21 (VDDA), C33.2, C34.2, C38.2, FB1.1
- net NFAULT: now reaches U1.25 (PB12)
- net INLA: now reaches U1.26 (PB13)
- net INLB: now reaches U1.27 (PB14)
- net INLC: now reaches U1.28 (PB15)
- net INHA: now reaches U1.30 (PA8)
- net INHB: now reaches U1.31 (PA9)
- net INHC: now reaches U1.32 (PA10)
- net USB_D-: now reaches U1.33 (PA11)
- net USB_D+: now reaches U1.34 (PA12)
- net SWDIO: now reaches U1.36 (PA13)
- net SWCLK: now reaches U1.37 (PA14)
- net at U1.39 (PC10): now also R23.1
- net at U1.40 (PC11): now also R24.1
- net SWO: now reaches U1.41 (PB3)
- net EN: now reaches U1.43 (PB5)
- net UART_TX: now reaches U1.44 (PB6)
- net UART_RX: now reaches U1.45 (PB7)
- net at U1.46 (PB8): now also R22.1
- net GND: now reaches U1.49 (VSS)
- net GND: now also C25.1, C26.1, C27.1, C28.1, C29.1, C30.1, C31.1, C32.1, C33.1, C34.1, C35.1, C36.1, C38.1, C9.1, D4.1 (K), D5.1 (K), R22.2, Y1.2 (G), Y1.4 (G)
- net at U1.5 (PF0): now also C27.2, Y1.1
- net at U1.6 (PF1): now also C28.2, Y1.3
- net NRST: now reaches U1.7 (PG10)
- net NRST: now also C36.2
- net at U1.8 (PA0): now also C29.2, R25.1
- net at U1.9 (PA1): now also C30.2, R26.1
- new net: D5.2 (A), R24.2
- new net: D4.2 (A), R23.2
- new net ISENSE_A: R25.2
- new net ISENSE_B: R26.2
- new net ISENSE_C: R27.2
- no-connect marks 0 -> 13
Other:
- note added: "Place as close as possible to VDDA and VREF"
- moved on the sheet: U1

Commit message: schematic completed
Parts:
- removed C25, C26, C36, C9: 100n, symbol Device:C
- added C37, C39, C40, C41: 100n, eCapacitor:0402, symbol Device:C
- C27, C28: value 15p -> 12p; footprint (none) -> eCapacitor:0402
- C29, C30, C31, C32, C33, C38: footprint (none) -> eCapacitor:0402
- C34: footprint (none) -> eCapacitor:0603
- C35: footprint (none) -> eCapacitor:0805
- D4, D5: footprint (none) -> eLED:0805_pol
- FB1: footprint (none) -> eResistor:0603
- R22, R23, R24, R25, R26, R27: footprint (none) -> eResistor:0402
- Y1: value 8Mhz -> 12Mhz; footprint (none) -> eCrystal:Crystal_SMD_ECX-32_Series_4Pin_3.2x2.5mm
Connections:
- net +3V3: now also C37.2, C39.2, C40.2
- net GND: now also C37.1, C39.1, C40.1, C41.1
- net NRST: now also C41.2
- net UART_RX: no longer names the net of U1.45 (PB7)
- net UART_TX: no longer names the net of U1.44 (PB6)
- no-connect marks 13 -> 15
Other:
- moved on the sheet: R22

Commit message: Schematic update, XT30/MR30 connectors and PCB layout in progress
- Connectors: AMASS XT30PW and MR30PW from Kicad_Libs (eConnector)
- Schematic updates on main, MCU and gate driver sheets
- PCB: footprints placed, routing in progress
Parts:
- D4, D5: footprint eLED:0805_pol -> eLED:0603_pol
Changed lines of the file:
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@@
 	(wire
 		(pts
+			(xy 45.72 46.99) (xy 45.72 48.26)
+		)
+		(stroke
+			(width 0)
+			(type default)
+		)
+	)
+	(wire
+		(pts
 			(xy 82.55 64.77) (xy 82.55 67.31)
 		)
@@
 	)
 	(symbol
+		(lib_id "ePowerSym:PWR_FLAG")
+		(at 45.72 46.99 0)
+		(unit 1)
+		(body_style 1)
+		(exclude_from_sim no)
+		(in_bom yes)
+		(on_board yes)
+		(in_pos_files yes)
+		(dnp no)
+		(fields_autoplaced yes)
+		(property "Reference" "#FLG04"
+			(at 45.72 45.085 0)
+			(hide yes)
+			(show_name no)
+			(do_not_autoplace no)
+			(effects
+				(font
+					(size 1.27 1.27)
+				)
+			)
+		)
+		(property "Value" "PWR_FLAG"
+			(at 45.72 41.91 0)
+			(hide yes)
+			(show_name no)
+			(do_not_autoplace no)
+			(effects
+				(font
+					(size 1.27 1.27)
+				)
+			)
+		)
+		(property "Footprint" ""
+			(at 45.72 46.99 0)
+			(hide yes)
+			(show_name no)
+			(do_not_autoplace no)
+			(effects
+				(font
+					(size 1.27 1.27)
+				)
+			)
+		)
+		(property "Datasheet" ""
+			(at 45.72 46.99 0)
+			(hide yes)
+			(show_name no)
+			(do_not_autoplace no)
+			(effects
+				(font
+					(size 1.27 1.27)
+				)
+			)
+		)
+		(property "Description" "Special symbol for telling ERC where power comes from"
+			(at 45.72 46.99 0)
+			(hide yes)
+			(show_name no)
+			(do_not_autoplace no)
+			(effects
+				(font
+					(size 1.27 1.27)
+				)
+			)
+		)
+		(pin "1"
+		)
+		(instances
+			(project "FOC_Driver"
+				(path "/56350f0b-fa2d-4452-8705-62cde497823d/d17cc26d-f1b1-46fa-8496-c55b233ba822"
+					(reference "#FLG04")
+					(unit 1)
+				)
+			)
+		)
+	)
+	(symbol
 		(lib_id "Device:R")
 		(at 233.68 77.47 90)
@@
 			)
 		)
-		(property "Footprint" "eLED:0805_pol"
+		(property "Footprint" "eLED:0603_pol"
 			(at 113.03 111.76 0)
 			(hide yes)
@@
 			)
 		)
-		(property "Footprint" "eLED:0805_pol"
+		(property "Footprint" "eLED:0603_pol"
 			(at 100.33 111.76 0)
 			(hide yes)

Commit message: Layout completed
Connections:
- net INHA: now also U1.32 (PA10); no longer U1.30 (PA8)
- net INHC: now also U1.30 (PA8); no longer U1.32 (PA10)
- net INLA: now also U1.28 (PB15); no longer U1.26 (PB13)
- net INLC: now also U1.26 (PB13); no longer U1.28 (PB15)
Changed lines of the file:
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@@
 		)
 	)
-	(hierarchical_label "INLC"
+	(hierarchical_label "INLA"
 		(shape output)
 		(at 125.73 148.59 180)
@@
 		)
 	)
-	(hierarchical_label "INHC"
+	(hierarchical_label "INHA"
 		(shape input)
 		(at 171.45 97.79 0)
@@
 		)
 	)
-	(hierarchical_label "INLA"
+	(hierarchical_label "INLC"
 		(shape output)
 		(at 125.73 143.51 180)
@@
 		)
 	)
-	(hierarchical_label "INHA"
-		(shape output)
+	(hierarchical_label "INHC"
+		(shape input)
 		(at 171.45 92.71 0)
 		(effects
